File: Hardware/RedVThingPlus.brd (EAGLE design)
At the start: 58.4 x 22.9 mm, 137 parts, among them J1 FEMALE 2x3, J2 USB Female Type C Connector, J4 QWIIC_RIGHT_ANGLE, Q1 3.1A/30V/105mΩ, U1 MCP73831, U2 AP2127K-1.8V, U3 AP2112-3.3V, U4 MK22FN128VLH10, U5 32MBit, U6 FE310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

Commit message: updating to 100 Ohm resistor on R8
Parts:
- R8: value 100k -> 100
Changed lines of the file:
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@@
 <attribute name="VALUE" x="48.895" y="6.096" size="0.6096" layer="27" font="vector" ratio="20" rot="R180" align="top-center"/>
 </element>
-<element name="R8" library="SparkFun-Resistors" package="0603" value="100k" x="48.895" y="6.858" smashed="yes">
+<element name="R8" library="SparkFun-Resistors" package="0603" value="100" x="48.895" y="6.858" smashed="yes">
 <attribute name="NAME" x="49.53" y="7.62" size="0.6096" layer="25" font="vector" ratio="20" align="bottom-center"/>
-<attribute name="PROD_ID" value="RES-07828" x="48.895" y="6.858" size="1.778" layer="27" display="off"/>
-<attribute name="VALUE" x="48.895" y="6.096" size="0.6096" layer="27" font="vector" ratio="20" align="top-center"/>
+<attribute name="PROD_ID" value="RES-07863" x="48.895" y="6.858" size="1.778" layer="27" display="off"/>
+<attribute name="VALUE" value="100" x="48.895" y="6.096" size="0.6096" layer="27" font="vector" ratio="20" align="top-center"/>
 </element>
 <element name="R9" library="SparkFun-Resistors" package="0603" value="4.7k" x="53.594" y="17.78" smashed="yes" rot="R270">
